Commit message: lidar

File: docker/create3_ws/src/create3_sim/irobot_create_common/irobot_create_description/urdf/create3.urdf.xacro (robot description, xacro)
@@ -11,4 +11,5 @@
   <xacro:include filename="$(find irobot_create_description)/urdf/sensors/optical_mouse.urdf.xacro"/>
   <xacro:include filename="$(find irobot_create_description)/urdf/wheel_with_wheeldrop.urdf.xacro" />
+  <xacro:include filename="$(find irobot_create_description)/urdf/sensors/lidar.urdf.xacro" />
   <!-- Gazebo version -->
   <xacro:arg name="gazebo"                       default="classic" />
@@ -86,4 +87,8 @@
     </inertial>
   </xacro:bumper>
+  <!-- LIDAR -->
+  <xacro:lidar2d_sensor name="lidar" parent="base_link">
+    <origin xyz="0 0 0.1" rpy="0 0 0"/>
+  </xacro:lidar2d_sensor>
   <!-- Wheels with mechanical wheel drop -->
   <xacro:wheel_with_wheeldrop name="left" gazebo="$(arg gazebo)" namespace="$(arg namespace)">

Commit message: Revert "lidar"
This reverts commit 13500a4eae372941b4c0ed096e0ef6bddf9f4359.

File: docker/create3_ws/src/create3_sim/irobot_create_common/irobot_create_description/urdf/create3.urdf.xacro (robot description, xacro)
@@ -11,5 +11,4 @@
   <xacro:include filename="$(find irobot_create_description)/urdf/sensors/optical_mouse.urdf.xacro"/>
   <xacro:include filename="$(find irobot_create_description)/urdf/wheel_with_wheeldrop.urdf.xacro" />
-  <xacro:include filename="$(find irobot_create_description)/urdf/sensors/lidar.urdf.xacro" />
   <!-- Gazebo version -->
   <xacro:arg name="gazebo"                       default="classic" />
@@ -87,8 +86,4 @@
     </inertial>
   </xacro:bumper>
-  <!-- LIDAR -->
-  <xacro:lidar2d_sensor name="lidar" parent="base_link">
-    <origin xyz="0 0 0.1" rpy="0 0 0"/>
-  </xacro:lidar2d_sensor>
   <!-- Wheels with mechanical wheel drop -->
   <xacro:wheel_with_wheeldrop name="left" gazebo="$(arg gazebo)" namespace="$(arg namespace)">

Commit message: Adding lidar simulation

File: docker/create3_ws/src/create3_sim/irobot_create_common/irobot_create_description/urdf/create3.urdf.xacro (robot description, xacro)
@@ -11,4 +11,5 @@
   <xacro:include filename="$(find irobot_create_description)/urdf/sensors/optical_mouse.urdf.xacro"/>
   <xacro:include filename="$(find irobot_create_description)/urdf/wheel_with_wheeldrop.urdf.xacro" />
+  <xacro:include filename="$(find irobot_create_description)/urdf/sensors/lidar.urdf.xacro"/>
   <!-- Gazebo version -->
   <xacro:arg name="gazebo"                       default="classic" />
@@ -129,4 +130,8 @@
     </gazebo>
   </xacro:if>
+  <!-- LIDAR -->
+  <xacro:lidar_2d name="lidar" gazebo="$(arg gazebo)" namespace="$(arg namespace)">
+    <origin xyz="0 0 0.06" rpy="0 0 0"/>
+  </xacro:lidar_2d>
   <!-- Mouse -->
   <xacro:optical_mouse gazebo="$(arg gazebo)" namespace="$(arg namespace)">

Commit message: lidar fix

File: docker/create3_ws/src/create3_sim/irobot_create_common/irobot_create_description/urdf/create3.urdf.xacro (robot description, xacro)
@@ -132,5 +132,5 @@
   <!-- LIDAR -->
   <xacro:lidar_2d name="lidar" gazebo="$(arg gazebo)" namespace="$(arg namespace)">
-    <origin xyz="0 0 0.06" rpy="0 0 0"/>
+    <origin xyz="0 0 0.12" rpy="0 0 0"/>
   </xacro:lidar_2d>
   <!-- Mouse -->

File: docker/create3_ws/src/create3_sim/irobot_create_common/irobot_create_description/urdf/sensors/lidar.urdf.xacro (robot description, xacro)
@@ -14,4 +14,10 @@
     <!-- Link -->
     <link name="${link_name}">
+      <visual>
+      <geometry>
+        <cylinder radius="0.02" length="0.05"/>
+      </geometry>
+      <material name="red"/>
+    </visual>
       <xacro:inertial_dummy/>
     </link>

Commit message: lidar fix

File: docker/create3_ws/src/create3_sim/irobot_create_common/irobot_create_description/urdf/create3.urdf.xacro (robot description, xacro)
@@ -268,5 +268,5 @@
     <gazebo>
       <plugin filename="libgz-sim-sensors-system.so" name="gz::sim::systems::Sensors">
-        <render_engine>ogre</render_engine>
+        <render_engine>ogre2</render_engine>
       </plugin>
     </gazebo>

File: docker/create3_ws/src/create3_sim/irobot_create_common/irobot_create_description/urdf/sensors/lidar.urdf.xacro (robot description, xacro)
@@ -27,9 +27,12 @@
     <!-- Ray sensor compatibile Classic/Ignition -->
     <gazebo reference="${link_name}">
+      <material>
+        <ambient>0 0 0 0</ambient>
+      </material>
       <xacro:ray_sensor sensor_name="${link_name}" gazebo="${gazebo}"
                         update_rate="${update_rate}" visualize="${visualize}"
                         h_samples="${h_samples}" h_res="1.0"
                         h_min_angle="-${fov/2}" h_max_angle="${fov/2}"
-                        v_samples="1" v_res="1.0" v_min_angle="0" v_max_angle="0"
+                        v_samples="1" v_res="1.0" v_min_angle="0.0" v_max_angle="0.0"
                         r_min="${min_range}" r_max="${max_range}" r_res="0.01">
         <plugin filename="libgazebo_ros_laser.so" name="${link_name}">
